File: ACTempDisconnect.kicad_sch (KiCad schematic)
At the start: 29 parts, among them J1001 Conn_01x03_Female, J1002 NTC_Connection, J1003 Conn_01x02_Female, J1004 Conn_01x03_Female, J1005 Conn_01x02_Female, K1001 ADW1103HLW, K1002 ADW1103HLW, K1003 ADW1103HLW, K1004 ADW1103HLW, U1001 LD03-23B03R2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

Commit message: Removed Neon from V2
Parts:
- removed NE1001: Lamp_Neon, Resistor_THT:R_Axial_DIN0204_L3.6mm_D1.6mm_P2.54mm_Vertical, symbol Device:Lamp_Neon
- removed R1001: 33k, Resistor_SMD:R_1206_3216Metric, symbol Device:R
Changed lines of the file:
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@@
-    (stroke (width 0) (type default) (color 0 0 0 0))
-  )
-  (wire (pts (xy 17.018 42.164) (xy 17.018 40.64))
     (stroke (width 0) (type default) (color 0 0 0 0))
   )
@@
     (effects (font (size 1.27 1.27)) (justify left bottom))
   )
-  (label "N_IN" (at 17.018 49.784 270)
-    (effects (font (size 1.27 1.27)) (justify right bottom))
-  )
   (label "NTC4" (at 264.668 96.266 180)
     (effects (font (size 1.27 1.27)) (justify right bottom))
@@
     (effects (font (size 1.27 1.27)) (justify right bottom))
   )
-  (label "_NEON" (at 17.018 41.402 0)
-    (effects (font (size 1.27 1.27)) (justify left bottom))
-  )
   (label "_AC_FUSE" (at 49.276 32.512 90)
     (effects (font (size 1.27 1.27)) (justify left bottom))
@@
   (label "NTC0" (at 265.176 106.426 180)
     (effects (font (size 1.27 1.27)) (justify right bottom))
-  )
-  (label "L_IN" (at 17.018 30.48 0)
-    (effects (font (size 1.27 1.27)) (justify left bottom))
   )
   (symbol (lib_id "ACTempDisconnect:DMHC4035LSD") (at 153.416 145.288 0) (unit 1)
@@
     (pin "2")
   )
-  (symbol (lib_id "Device:R") (at 17.018 45.974 0) (unit 1)
-    (in_bom yes) (on_board yes) (fields_autoplaced)
-    (property "Reference" "R1001" (id 0) (at 18.796 45.1393 0)
-      (effects (font (size 1.27 1.27)) (justify left))
-    )
-    (property "Value" "33k" (id 1) (at 18.796 47.6762 0)
-      (effects (font (size 1.27 1.27)) (justify left))
-    )
-    (property "Footprint" "Resistor_SMD:R_1206_3216Metric" (id 2) (at 15.24 45.974 90)
-      (effects (font (size 1.27 1.27)) hide)
-    )
-    (property "Datasheet" "~" (id 3) (at 17.018 45.974 0)
-      (effects (font (size 1.27 1.27)) hide)
-    )
-    (pin "1")
-    (pin "2")
-  )
   (symbol (lib_id "power:+3V3") (at 149.606 124.968 0) (unit 1)
     (in_bom yes) (on_board yes) (fields_autoplaced)
@@
     (pin "3")
   )
-  (symbol (lib_id "Device:Lamp_Neon") (at 17.018 35.56 0) (unit 1)
-    (in_bom yes) (on_board yes) (fields_autoplaced)
-    (property "Reference" "NE1001" (id 0) (at 20.193 34.7253 0)
-      (effects (font (size 1.27 1.27)) (justify left))
-    )
-    (property "Value" "Lamp_Neon" (id 1) (at 20.193 37.2622 0)
-      (effects (font (size 1.27 1.27)) (justify left))
-    )
-    (property "Footprint" "Resistor_THT:R_Axial_DIN0204_L3.6mm_D1.6mm_P2.54mm_Vertical" (id 2) (at 17.018 33.02 90)
-      (effects (font (size 1.27 1.27)) hide)
-    )
-    (property "Datasheet" "https://www.mouser.com/datasheet/2/244/GT-NE4H1125T-80186.pdf" (id 3) (at 17.018 33.02 90)
-      (effects (font (size 1.27 1.27)) hide)
-    )
-    (property "MPN" "GT-NE4H1125T " (id 4) (at 17.018 35.56 0)
-      (effects (font (size 1.27 1.27)) hide)
-    )
-    (pin "1")
-    (pin "2")
-  )
   (symbol (lib_id "ACTempDisconnect:WP934SA") (at 28.956 62.992 0) (unit 1)
     (in_bom yes) (on_board yes) (fields_autoplaced)
@@
       (reference "LED1001") (unit 1) (value "WP934SA") (footprint "Library:WP934SA_LILYLGD")
     )
-    (path "/edf5211f-0056-4645-8540-c4593f45f518"
-      (reference "NE1001") (unit 1) (value "Lamp_Neon") (footprint "Resistor_THT:R_Axial_DIN0204_L3.6mm_D1.6mm_P2.54mm_Vertical")
-    )
-    (path "/ad520c33-4a65-49f8-abd7-ff8d24d6bed1"
-      (reference "R1001") (unit 1) (value "33k") (footprint "Resistor_SMD:R_1206_3216Metric")
-    )
     (path "/751eee74-c170-475a-80ff-72207ed2354a"

Commit message: Rev 2
Simplified the layout. Reduced down to 2 layers.
Added top/bottom traces to split the current.
Parts:
- removed C1005: 2.2u, Capacitor_SMD:C_0805_2012Metric_Pad1.18x1.45mm_HandSolder, symbol Device:C
- removed K1003: ADW1103HLW, Relay_THT:Relay_1P1T_NO_10x24x18.8mm_Panasonic_ADW11xxxxW_THT, symbol Relay:ADW11
- removed U1004: DMHC4035LSD, Package_SO:SOIC-8_3.9x4.9mm_P1.27mm, symbol ACTempDisconnect:DMHC4035LSD
- J1001: MPN OSTT7030150 -> (none)
Connections:
- net N_OUT is gone; now on net N_IN: J1004.1 (Pin_1)
- net L_HEATER0: now also J1003.1 (Pin_1); no longer J1003.2 (Pin_2)
- net L_HEATER1: now also J1003.2 (Pin_2); no longer J1003.1 (Pin_1)

Commit message: 8 to 4 NTC
Reduced down from 8 to 4 NTCs, for cost down and packaging
considerations.
Parts:
- removed J1002: NTC_Connection, Library:736-108, symbol Connector_Generic:Conn_02x08_Top_Bottom
- removed RN1001: R_Pack08, Package_SO:SOIC-16_3.9x9.9mm_P1.27mm, symbol Device:R_Pack08
- added J1002: Conn_02x04_Counter_Clockwise, Library:736-104, symbol Connector_Generic:Conn_02x04_Counter_Clockwise
- added RN1001: R_Pack04, Resistor_SMD:R_Array_Convex_4x1206, symbol Device:R_Pack04
Connections:
- net +3V3: now also RN1001.1 (R1.1), RN1001.2 (R2.1), RN1001.3 (R3.1), RN1001.4 (R4.1)
- net GND: now also J1002.5 (Pin_5), J1002.6 (Pin_6), J1002.7 (Pin_7), J1002.8 (Pin_8)
- net NTC0: now also J1002.1 (Pin_1), RN1001.8 (R1.2)
- net NTC1: now also J1002.2 (Pin_2), RN1001.7 (R2.2)
- net NTC2: now also J1002.3 (Pin_3), RN1001.6 (R3.2)
- net NTC3: now also J1002.4 (Pin_4), RN1001.5 (R4.2)
Other:
- sheet MCU ports: added NTC[0..3]; removed NTC[0..7]
