File: MCU.kicad_sch (KiCad schematic)
At the start: 20 parts, among them J2001 TAG_CONNECT, U2001 STM32F030K6Tx, U2003 24FC01T

Commit message: Rev 2
Simplified the layout. Reduced down to 2 layers.
Added top/bottom traces to split the current.
Parts:
- removed TP2011, TP2012, TP2013, TP2014, TP2015, TP2016: TestPoint, TestPoint:TestPoint_Pad_D1.0mm, symbol Connector:TestPoint
Connections:
- net CHARGE_RELAY+: now also U2001.25 (PA15); no longer U2001.26 (PB3)
- net CHARGE_RELAY-: now also U2001.26 (PB3); no longer U2001.27 (PB4)
- net G: now also U2001.18 (PA8); no longer U2001.22 (PA12)
- net HEAT_RELAY_0+: now also U2001.28 (PB5); no longer U2001.2 (PF0)
- net HEAT_RELAY_0-: now also U2001.27 (PB4); no longer U2001.3 (PF1)
- net HEAT_RELAY_1+: now also U2001.3 (PF1); no longer U2001.21 (PA11)
- net HEAT_RELAY_1-: now also U2001.2 (PF0); no longer U2001.18 (PA8)
- no-connect marks 2 -> 0
Changed lines of the file:
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@@
   (junction (at 52.07 123.19) (diameter 0) (color 0 0 0 0)
   )
-  (no_connect (at 66.04 167.894))
-  (no_connect (at 38.1 162.814))
   (bus_entry (at 260.858 29.972) (size -2.54 2.54)
     (stroke (width 0) (type default) (color 0 0 0 0))
@@
     (stroke (width 0) (type default) (color 0 0 0 0))
   )
+  (label "RELAY_CHARGE-" (at 38.1 157.734 180)
+    (effects (font (size 1.27 1.27)) (justify right bottom))
+  )
   (label "UART_RX" (at 38.354 103.378 0)
     (effects (font (size 1.27 1.27)) (justify left bottom))
@@
     (effects (font (size 1.27 1.27)) (justify right bottom))
   )
-  (label "RELAY_CHARGE+" (at 38.1 157.734 180)
-    (effects (font (size 1.27 1.27)) (justify right bottom))
-  )
-  (label "RELAY_CHARGE+" (at 199.39 74.168 180)
-    (effects (font (size 1.27 1.27)) (justify right bottom))
-  )
   (label "NTC6" (at 66.04 145.034 0)
     (effects (font (size 1.27 1.27)) (justify left bottom))
@@
     (effects (font (size 1.27 1.27)) (justify right bottom))
   )
-  (label "HRELAY1-" (at 66.04 150.114 0)
-    (effects (font (size 1.27 1.27)) (justify left bottom))
+  (label "HRELAY0-" (at 38.1 160.274 180)
+    (effects (font (size 1.27 1.27)) (justify right bottom))
   )
   (label "UART_RX" (at 138.43 110.744 180)
@@
     (effects (font (size 1.27 1.27)) (justify left bottom))
   )
-  (label "HRELAY0-" (at 199.39 88.9 180)
-    (effects (font (size 1.27 1.27)) (justify right bottom))
-  )
   (label "NTC1" (at 263.652 34.29 270)
     (effects (font (size 1.27 1.27)) (justify right bottom))
@@
     (effects (font (size 1.27 1.27)) (justify left bottom))
   )
+  (label "HRELAY0+" (at 38.1 162.814 180)
+    (effects (font (size 1.27 1.27)) (justify right bottom))
+  )
   (label "MCU_RX" (at 134.62 91.694 180)
     (effects (font (size 1.27 1.27)) (justify right bottom))
   )
+  (label "HRELAY1-" (at 38.1 145.034 180)
+    (effects (font (size 1.27 1.27)) (justify right bottom))
+  )
   (label "HRELAY0+" (at 267.716 18.542 180)
     (effects (font (size 1.27 1.27)) (justify right bottom))
@@
     (effects (font (size 1.27 1.27)) (justify right bottom))
   )
-  (label "G" (at 66.04 160.274 0)
+  (label "G" (at 66.04 150.114 0)
     (effects (font (size 1.27 1.27)) (justify left bottom))
   )
@@
     (effects (font (size 1.27 1.27)) (justify right bottom))
   )
-  (label "HRELAY1+" (at 66.04 157.734 0)
-    (effects (font (size 1.27 1.27)) (justify left bottom))
-  )
   (label "VDDA" (at 55.88 124.714 0)
     (effects (font (size 1.27 1.27)) (justify left bottom))
@@
     (effects (font (size 1.27 1.27)) (justify left bottom))
   )
-  (label "HRELAY0+" (at 38.1 145.034 180)
-    (effects (font (size 1.27 1.27)) (justify right bottom))
-  )
-  (label "RELAY_CHARGE-" (at 199.39 78.994 180)
-    (effects (font (size 1.27 1.27)) (justify right bottom))
-  )
   (label "NTC0" (at 66.04 129.794 0)
     (effects (font (size 1.27 1.27)) (justify left bottom))
@@
     (effects (font (size 1.27 1.27)) (justify right bottom))
   )
+  (label "HRELAY1+" (at 38.1 147.574 180)
+    (effects (font (size 1.27 1.27)) (justify right bottom))
+  )
   (label "I2C_SDA" (at 126.238 169.418 180)
     (effects (font (size 1.27 1.27)) (justify right bottom))
   )
-  (label "HRELAY1-" (at 199.39 99.568 180)
-    (effects (font (size 1.27 1.27)) (justify right bottom))
-  )
   (label "NTC3" (at 66.04 137.414 0)
     (effects (font (size 1.27 1.27)) (justify left bottom))
   )
-  (label "HRELAY0+" (at 199.39 83.82 180)
-    (effects (font (size 1.27 1.27)) (justify right bottom))
-  )
   (label "NTC0" (at 265.176 34.29 270)
     (effects (font (size 1.27 1.27)) (justify right bottom))
@@
     (effects (font (size 1.27 1.27)) (justify left bottom))
   )
-  (label "HRELAY0-" (at 38.1 147.574 180)
-    (effects (font (size 1.27 1.27)) (justify right bottom))
-  )
   (label "SWDCLK" (at 66.04 165.354 0)
     (effects (font (size 1.27 1.27)) (justify left bottom))
@@
     (effects (font (size 1.27 1.27)) (justify right bottom))
   )
-  (label "HRELAY1+" (at 199.39 94.234 180)
-    (effects (font (size 1.27 1.27)) (justify right bottom))
-  )
   (label "NTC2" (at 66.04 134.874 0)
     (effects (font (size 1.27 1.27)) (justify left bottom))
@@
     (effects (font (size 1.27 1.27)) (justify left bottom))
   )
-  (label "RELAY_CHARGE-" (at 38.1 160.274 180)
-    (effects (font (size 1.27 1.27)) (justify right bottom))
+  (label "RELAY_CHARGE+" (at 66.04 167.894 0)
+    (effects (font (size 1.27 1.27)) (justify left bottom))
   )
   (label "I2C_SCL" (at 88.138 186.182 180)
@@
     (pin "1")
   )
-  (symbol (lib_id "Connector:TestPoint") (at 199.39 74.168 0) (unit 1)
-    (in_bom yes) (on_board yes) (fields_autoplaced)
-    (property "Reference" "TP2011" (id 0) (at 200.787 70.0313 0)
-      (effects (font (size 1.27 1.27)) (justify left))
-    )
-    (property "Value" "TestPoint" (id 1) (at 200.787 72.5682 0)
-      (effects (font (size 1.27 1.27)) (justify left))
-    )
-    (property "Footprint" "TestPoint:TestPoint_Pad_D1.0mm" (id 2) (at 204.47 74.168 0)
-      (effects (font (size 1.27 1.27)) hide)
-    )
-    (property "Datasheet" "~" (id 3) (at 204.47 74.168 0)
-      (effects (font (size 1.27 1.27)) hide)
-    )
-    (pin "1")
-  )
   (symbol (lib_id "power:GND") (at 83.058 78.486 0) (unit 1)
     (in_bom yes) (on_board yes) (fields_autoplaced)
@@
     )
     (property "Datasheet" "" (id 3) (at 83.058 78.486 0)
-      (effects (font (size 1.27 1.27)) hide)
-    )
-    (pin "1")
-  )
-  (symbol (lib_id "Connector:TestPoint") (at 199.39 78.994 0) (unit 1)
-    (in_bom yes) (on_board yes) (fields_autoplaced)
-    (property "Reference" "TP2012" (id 0) (at 200.787 74.8573 0)
-      (effects (font (size 1.27 1.27)) (justify left))
-    )
-    (property "Value" "TestPoint" (id 1) (at 200.787 77.3942 0)
-      (effects (font (size 1.27 1.27)) (justify left))
-    )
-    (property "Footprint" "TestPoint:TestPoint_Pad_D1.0mm" (id 2) (at 204.47 78.994 0)
-      (effects (font (size 1.27 1.27)) hide)
-    )
-    (property "Datasheet" "~" (id 3) (at 204.47 78.994 0)
       (effects (font (size 1.27 1.27)) hide)
     )
@@
     (pin "3")
   )
-  (symbol (lib_id "Connector:TestPoint") (at 199.39 83.82 0) (unit 1)
-    (in_bom yes) (on_board yes) (fields_autoplaced)
-    (property "Reference" "TP2013" (id 0) (at 200.787 79.6833 0)
-      (effects (font (size 1.27 1.27)) (justify left))
-    )
-    (property "Value" "TestPoint" (id 1) (at 200.787 82.2202 0)
-      (effects (font (size 1.27 1.27)) (justify left))
-    )
-    (property "Footprint" "TestPoint:TestPoint_Pad_D1.0mm" (id 2) (at 204.47 83.82 0)
-      (effects (font (size 1.27 1.27)) hide)
-    )
-    (property "Datasheet" "~" (id 3) (at 204.47 83.82 0)
-      (effects (font (size 1.27 1.27)) hide)
-    )
-    (pin "1")
-  )
   (symbol (lib_id "Device:R") (at 126.238 165.608 0) (unit 1)
     (in_bom yes) (on_board yes) (fields_autoplaced)
@@
     (pin "1")
   )
-  (symbol (lib_id "Connector:TestPoint") (at 199.39 99.568 0) (unit 1)
-    (in_bom yes) (on_board yes) (fields_autoplaced)
-    (property "Reference" "TP2016" (id 0) (at 200.787 95.4313 0)
-      (effects (font (size 1.27 1.27)) (justify left))
-    )
-    (property "Value" "TestPoint" (id 1) (at 200.787 97.9682 0)
-      (effects (font (size 1.27 1.27)) (justify left))
-    )
-    (property "Footprint" "TestPoint:TestPoint_Pad_D1.0mm" (id 2) (at 204.47 99.568 0)
-      (effects (font (size 1.27 1.27)) hide)
-    )
-    (property "Datasheet" "~" (id 3) (at 204.47 99.568 0)
-      (effects (font (size 1.27 1.27)) hide)
-    )
-    (pin "1")
-  )
   (symbol (lib_id "power:+3V3") (at 40.64 92.71 0) (unit 1)
     (in_bom yes) (on_board yes) (fields_autoplaced)
@@
     (pin "1")
     (pin "2")
-  )
-  (symbol (lib_id "Connector:TestPoint") (at 199.39 88.9 0) (unit 1)
-    (in_bom yes) (on_board yes) (fields_autoplaced)
-    (property "Reference" "TP2014" (id 0) (at 200.787 84.7633 0)
-      (effects (font (size 1.27 1.27)) (justify left))
-    )
-    (property "Value" "TestPoint" (id 1) (at 200.787 87.3002 0)
-      (effects (font (size 1.27 1.27)) (justify left))
-    )
-    (property "Footprint" "TestPoint:TestPoint_Pad_D1.0mm" (id 2) (at 204.47 88.9 0)
-      (effects (font (size 1.27 1.27)) hide)
-    )
-    (property "Datasheet" "~" (id 3) (at 204.47 88.9 0)
-      (effects (font (size 1.27 1.27)) hide)
-    )
-    (pin "1")
   )
   (symbol (lib_id "power:+3V3") (at 83.058 70.866 0) (unit 1)
@@
     (pin "5")
   )
-  (symbol (lib_id "Connector:TestPoint") (at 199.39 94.234 0) (unit 1)
-    (in_bom yes) (on_board yes) (fields_autoplaced)
-    (property "Reference" "TP2015" (id 0) (at 200.787 90.0973 0)
-      (effects (font (size 1.27 1.27)) (justify left))
-    )
-    (property "Value" "TestPoint" (id 1) (at 200.787 92.6342 0)
-      (effects (font (size 1.27 1.27)) (justify left))
-    )
-    (property "Footprint" "TestPoint:TestPoint_Pad_D1.0mm" (id 2) (at 204.47 94.234 0)
-      (effects (font (size 1.27 1.27)) hide)
-    )
-    (property "Datasheet" "~" (id 3) (at 204.47 94.234 0)
-      (effects (font (size 1.27 1.27)) hide)
-    )
-    (pin "1")
-  )
   (symbol (lib_id "MCU_ST_STM32F0:STM32F030K6Tx") (at 53.34 147.574 0) (unit 1)

Commit message: 8 to 4 NTC
Reduced down from 8 to 4 NTCs, for cost down and packaging
considerations.
Connections:
- net NTC4: no longer names the net of U2001.10 (PA4)
- net NTC5: no longer names the net of U2001.11 (PA5)
- net NTC6: no longer names the net of U2001.12 (PA6)
- net NTC7: no longer names the net of U2001.13 (PA7)
- no-connect marks 0 -> 4
Changed lines of the file:
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@@
   (junction (at 52.07 123.19) (diameter 0) (color 0 0 0 0)
   )
-  (bus_entry (at 260.858 29.972) (size -2.54 2.54)
-    (stroke (width 0) (type default) (color 0 0 0 0))
-  )
-  (bus_entry (at 259.588 29.972) (size -2.54 2.54)
-    (stroke (width 0) (type default) (color 0 0 0 0))
-  )
-  (bus_entry (at 258.318 29.972) (size -2.54 2.54)
-    (stroke (width 0) (type default) (color 0 0 0 0))
-  )
+  (no_connect (at 66.04 147.574))
+  (no_connect (at 66.04 145.034))
+  (no_connect (at 66.04 142.494))
+  (no_connect (at 66.04 139.954))
   (bus_entry (at 264.668 29.972) (size -2.54 2.54)
     (stroke (width 0) (type default) (color 0 0 0 0))
@@
     (stroke (width 0) (type default) (color 0 0 0 0))
   )
-  (bus_entry (at 262.128 29.972) (size -2.54 2.54)
-    (stroke (width 0) (type default) (color 0 0 0 0))
-  )
   (bus_entry (at 263.398 29.972) (size -2.54 2.54)
     (stroke (width 0) (type default) (color 0 0 0 0))
@@
     (stroke (width 0) (type default) (color 0 0 0 0))
   )
-  (wire (pts (xy 255.778 32.512) (xy 254.508 32.512))
-    (stroke (width 0) (type default) (color 0 0 0 0))
-  )
   (wire (pts (xy 49.53 100.838) (xy 49.53 101.6))
     (stroke (width 0) (type default) (color 0 0 0 0))
   )
-  (bus (pts (xy 260.858 29.972) (xy 262.128 29.972))
-    (stroke (width 0) (type default) (color 0 0 0 0))
-  )
-  (wire (pts (xy 259.588 34.29) (xy 259.08 34.29))
-    (stroke (width 0) (type default) (color 0 0 0 0))
-  )
   (wire (pts (xy 113.538 183.896) (xy 116.078 183.896))
     (stroke (width 0) (type default) (color 0 0 0 0))
@@
     (stroke (width 0) (type default) (color 0 0 0 0))
   )
-  (bus (pts (xy 257.556 29.972) (xy 258.318 29.972))
-    (stroke (width 0) (type default) (color 0 0 0 0))
-  )
   (wire (pts (xy 260.858 34.29) (xy 260.604 34.29))
     (stroke (width 0) (type default) (color 0 0 0 0))
@@
     (stroke (width 0) (type default) (color 0 0 0 0))
   )
-  (wire (pts (xy 258.318 32.512) (xy 258.318 34.29))
-    (stroke (width 0) (type default) (color 0 0 0 0))
-  )
   (wire (pts (xy 33.782 121.92) (xy 33.782 121.412))
     (stroke (width 0) (type default) (color 0 0 0 0))
@@
     (stroke (width 0) (type default) (color 0 0 0 0))
   )
-  (wire (pts (xy 254.508 32.512) (xy 254.508 34.29))
-    (stroke (width 0) (type default) (color 0 0 0 0))
-  )
   (wire (pts (xy 53.34 173.99) (xy 53.34 172.974))
     (stroke (width 0) (type default) (color 0 0 0 0))
@@
     (stroke (width 0) (type default) (color 0 0 0 0))
   )
-  (wire (pts (xy 258.318 34.29) (xy 257.556 34.29))
-    (stroke (width 0) (type default) (color 0 0 0 0))
-  )
   (wire (pts (xy 33.782 129.54) (xy 33.782 129.794))
     (stroke (width 0) (type default) (color 0 0 0 0))
   )
-  (wire (pts (xy 256.032 34.29) (xy 257.048 34.29))
-    (stroke (width 0) (type default) (color 0 0 0 0))
-  )
-  (bus (pts (xy 259.588 29.972) (xy 260.858 29.972))
-    (stroke (width 0) (type default) (color 0 0 0 0))
-  )
   (wire (pts (xy 105.918 191.262) (xy 111.506 191.262))
     (stroke (width 0) (type default) (color 0 0 0 0))
@@
     (stroke (width 0) (type default) (color 0 0 0 0))
   )
-  (wire (pts (xy 257.048 32.512) (xy 257.048 34.29))
-    (stroke (width 0) (type default) (color 0 0 0 0))
-  )
   (wire (pts (xy 263.398 32.512) (xy 263.398 34.29))
     (stroke (width 0) (type default) (color 0 0 0 0))
@@
     (stroke (width 0) (type default) (color 0 0 0 0))
   )
-  (wire (pts (xy 259.588 32.512) (xy 259.588 34.29))
-    (stroke (width 0) (type default) (color 0 0 0 0))
-  )
   (wire (pts (xy 147.066 70.104) (xy 151.13 70.104))
     (stroke (width 0) (type default) (color 0 0 0 0))
@@
     (stroke (width 0) (type default) (color 0 0 0 0))
   )
-  (bus (pts (xy 258.318 29.972) (xy 259.588 29.972))
-    (stroke (width 0) (type default) (color 0 0 0 0))
-  )
   (wire (pts (xy 111.506 191.262) (xy 111.506 191.008))
     (stroke (width 0) (type default) (color 0 0 0 0))
@@
     (effects (font (size 1.27 1.27)) (justify right bottom))
   )
-  (label "NTC6" (at 66.04 145.034 0)
-    (effects (font (size 1.27 1.27)) (justify left bottom))
-  )
-  (label "NTC7" (at 254.508 34.29 270)
-    (effects (font (size 1.27 1.27)) (justify right bottom))
-  )
   (label "MCU_TX" (at 134.62 105.664 180)
     (effects (font (size 1.27 1.27)) (justify right bottom))
@@
     (effects (font (size 1.27 1.27)) (justify left bottom))
   )
-  (label "NTC4" (at 66.04 139.954 0)
-    (effects (font (size 1.27 1.27)) (justify left bottom))
-  )
-  (label "NTC6" (at 256.032 34.29 270)
-    (effects (font (size 1.27 1.27)) (justify right bottom))
-  )
   (label "G" (at 66.04 150.114 0)
     (effects (font (size 1.27 1.27)) (justify left bottom))
@@
     (effects (font (size 1.27 1.27)) (justify left bottom))
   )
-  (label "NTC5" (at 66.04 142.494 0)
-    (effects (font (size 1.27 1.27)) (justify left bottom))
-  )
   (label "NTC0" (at 66.04 129.794 0)
     (effects (font (size 1.27 1.27)) (justify left bottom))
@@
     (effects (font (size 1.27 1.27)) (justify left bottom))
   )
-  (label "NTC7" (at 66.04 147.574 0)
-    (effects (font (size 1.27 1.27)) (justify left bottom))
-  )
   (label "HRELAY1+" (at 267.716 22.86 180)
     (effects (font (size 1.27 1.27)) (justify right bottom))
@@
     (effects (font (size 1.27 1.27)) (justify left bottom))
   )
-  (label "NTC4" (at 259.08 34.29 270)
-    (effects (font (size 1.27 1.27)) (justify right bottom))
-  )
   (label "NTC2" (at 66.04 134.874 0)
     (effects (font (size 1.27 1.27)) (justify left bottom))
   )
-  (label "NTC5" (at 257.556 34.29 270)
-    (effects (font (size 1.27 1.27)) (justify right bottom))
-  )
   (label "SWDIO" (at 38.354 108.458 0)
     (effects (font (size 1.27 1.27)) (justify left bottom))
@@
     (effects (font (size 1.27 1.27)) (justify left))
   )
-  (hierarchical_label "NTC[0..7]" (shape input) (at 267.716 29.972 0)
-    (effects (font (size 1.27 1.27)) (justify left))
-  )
+  (hierarchical_label "NTC[0..3]" (shape input) (at 267.716 29.972 0)
+    (effects (font (size 1.27 1.27)) (justify left))
+  )
